File: hardware/airnote.kicad_pcb (KiCad board)
At the start: 4 copper layers, 90 x 70 mm, 73 parts, among them J1 USB-C USB2.0, J2 SWD 3V3 GND DIO CLK RUN, J3 SPEAKER 8ohm >=1W, SW1 BOOTSEL, SW2 RESET, SW3 MUTE / PLAY, U1 RP2040, U2 W25Q16JVSSIQ, U3 AP2112K-3.3, U4 VL53L1CXV0FY/1, U5 MAX98357AETE+T, Y1 12MHz ABM8-272-T3

Commit message: Phase 2: rev 0.2 layout with coupled USB pair, crystal/IOVDD fixes and JLC sourcing
Hardware (implementer, verified by overseer):
- Stackup set to JLC04161H-7628. USB_DIFF net class at 0.25/0.15 mm; all six
  USB nets on F.Cu with no vias over continuous In1 GND.
- Crystal moved under U1: XIN 4.1 mm with no vias (was 7.8 mm, 2 vias).
  IOVDD pin 22 to C6 2.9 mm (was 6.1 mm).
- airnote.kicad_dru values now carry units. KiCad had been discarding the
  unitless file, so its rules were never enforced. DRC still passes.
- U2 corrected to W25Q16JVSNIQ (150-mil, matches footprint). J1, RV1, J2 and
  passives switched to in-stock JLC/LCSC parts. LCSC numbers in the schematic,
  footprints and bom.csv.
- Three global fiducials. ERC 0, DRC 0, parity 0; outputs regenerated.

Docs: fabrication plan, requirements, README, assembly brief and bring-up
updated for rev 0.2. Surface finish recorded as an order-time decision.
Parts:
- added FID1: Fiducial, Fiducial:Fiducial_1mm_Mask2mm, F.Cu at (53.5, 61.5)
- added FID2: Fiducial, Fiducial:Fiducial_1mm_Mask2mm, F.Cu at (61.5, 116.5)
- added FID3: Fiducial, Fiducial:Fiducial_1mm_Mask2mm, F.Cu at (130.0, 53.5)
- U2: value W25Q16JVSSIQ -> W25Q16JVSNIQ
- moved C1 4.04 mm to (86.7, 90.4), turned to -90 degrees
- moved C2 3.27 mm to (91.9, 92.6), turned to -90 degrees
- moved D1 3.23 mm to (71.1, 65.1), turned to 90 degrees
- moved Y1 2.69 mm to (89.3, 91.5), turned to -90 degrees
- moved R1 2.48 mm to (89.7, 87.7), turned to -90 degrees
- moved C11 1.98 mm to (92.4, 87.0), turned to 0 degrees
- moved C6 1.74 mm to (92.0, 88.5)
- moved R9 1.00 mm to (92.6, 74.3)
- moved R8 0.45 mm to (91.0, 73.6)
Routing:
- net USB_DP_ESD: track 24.1 -> 44.5 mm, vias 2 -> 0
- net SENSOR_XSHUT: track 50.8 -> 60.2 mm
- net USB_DM_ESD: track 34.4 -> 42.2 mm
- net +1V1: track 32.0 -> 25.3 mm
- net XOUT: track 6.40 -> 0.80 mm
- net XIN: track 10.5 -> 5.18 mm, vias 2 -> 0
- net XTAL_OUT: track 9.65 -> 4.96 mm
- net +3V3: track 223.4 -> 219.2 mm, vias 9 -> 8
- net GND: track 15.9 -> 19.8 mm, vias 34 -> 39
- net USB_DP: track 19.7 -> 17.1 mm
- net USB_DM: track 20.3 -> 18.5 mm, vias 2 -> 0
- net BOOTSEL_SW: track 18.5 -> 16.9 mm, vias 0 -> 2
- net VBUS_RAW: track 35.9 -> 34.3 mm, vias 0 -> 2
- net CC1: track 11.1 -> 12.5 mm, vias 0 -> 2
- net QSPI_D0: track 10.6 -> 9.58 mm

Commit message: Phase 4: rev 0.2 review fixes and JLC order package
Fixes for the independent review of 78444e8:
- MFG-05: removed the GND via 0.133 mm from J1 shell slot S1. No drill web
  on the board is now below JLC's minimums (reviews/inspect_layout.py: 23/23).
- MFG-11: silkscreen and all title blocks at rev 0.2 (gerber job Revision
  0.2); export README rewritten. Copper finish stays an order-form choice.
- +5V after F1 widened from 0.15 to 0.4 mm, with a parallel via at U5
  (about 0.31 to 0.12 ohm to U5).
- C15 GND via moved out of the pad. hardware/README USB figures corrected to
  the reviewer's measurements.

Order package, generated and hashed by export_outputs.py:
airnote-jlc-bom.csv (26 lines, 58 parts), airnote-jlc-cpl.csv (58 parts,
KiCad rotations, no correction table), airnote-jlc-gerbers.zip, a
JLCJLCJLCJLC order-number marker on B.Silkscreen, and upload steps.

ERC 0, DRC 0, parity 0. Overseer dispositions of the review concerns are in
docs/fabrication_plan.md.
Routing:
- net +5V: track 140.0 -> 141.9 mm, vias 2 -> 3
- net GND: track 19.8 -> 19.9 mm, vias 39 -> 38
Other:
- board text added: "JLCJLCJLCJLC"
- board text added: "v0.2 ENGINEERING PROTOTYPE"
- board text removed: "v0.1 ENGINEERING PROTOTYPE"
Changed lines of the file:
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@@
 	)
 	(paper "A4")
+	(title_block
+		(title "AirNote")
+		(date "2026-10-10")
+		(rev "0.2")
+		(company "AirNote side project")
+	)
 	(layers
 		(0 "F.Cu" signal)
@@
 				(type "Top Solder Mask")
 				(thickness 0.01)
-				(epsilon_r 3.8)
-				(loss_tangent 0)
 			)
 			(layer "F.Cu"
@@
 				(type "Bottom Solder Mask")
 				(thickness 0.01)
-				(epsilon_r 3.8)
-				(loss_tangent 0)
 			)
 			(layer "B.Paste"
@@
 		)
 	)
-	(gr_text "v0.1 ENGINEERING PROTOTYPE"
+	(gr_text "v0.2 ENGINEERING PROTOTYPE"
 		(at 80 97 0)
 		(layer "F.SilkS")
@@
 		)
 	)
+	(gr_text "JLCJLCJLCJLC"
+		(at 70 90 0)
+		(layer "B.SilkS")
+		(effects
+			(font
+				(size 1 0.9)
+				(thickness 0.15)
+			)
+			(justify mirror)
+		)
+	)
 	(segment
 		(start 91.8 77.125)
@@
 	)
 	(segment
-		(start 118.7076 103.9298)
-		(end 119.5452 103.9298)
-		(width 0.15)
+		(start 112.9 59.292)
+		(end 113.55 59.942)
+		(width 0.4)
 		(layer "F.Cu")
 		(net 3)
@@
 	)
 	(segment
-		(start 119.25 102.425)
-		(end 119.25 103.725)
-		(width 0.3)
-		(locked yes)
+		(start 121.225 103.975)
+		(end 121.45 103.8)
+		(width 0.4)
 		(layer "F.Cu")
 		(net 3)
 	)
 	(segment
-		(start 58.9717 55.9397)
-		(end 60.8114 54.1)
-		(width 0.15)
+		(start 70.175 70.05)
+		(end 72.862 70.05)
+		(width 0.4)
 		(layer "F.Cu")
 		(net 3)
 	)
 	(segment
-		(start 119.5 103.975)
-		(end 121.225 103.975)
+		(start 61.4 67)
+		(end 68 67)
+		(width 0.4)
+		(layer "F.Cu")
+		(net 3)
+	)
+	(segment
+		(start 119.25 102.425)
+		(end 119.25 103.725)
 		(width 0.3)
 		(locked yes)
@@
 	)
 	(segment
-		(start 70.175 69.175)
-		(end 68 67)
-		(width 0.15)
+		(start 58.8 55.9)
+		(end 58.8 64.4)
+		(width 0.4)
 		(layer "F.Cu")
 		(net 3)
@@
 	)
 	(segment
-		(start 58.9717 64.3697)
-		(end 58.9717 55.9397)
-		(width 0.15)
-		(layer "F.Cu")
-		(net 3)
-	)
-	(segment
-		(start 70.175 70.05)
+		(start 68 67)
 		(end 70.175 69.175)
-		(width 0.15)
+		(width 0.4)
 		(layer "F.Cu")
 		(net 3)
 	)
 	(segment
-		(start 70.75 54.1)
-		(end 100.8627 54.1)
-		(width 0.15)
+		(start 58.8 64.4)
+		(end 61.4 67)
+		(width 0.4)
 		(layer "F.Cu")
 		(net 3)
 	)
 	(segment
-		(start 121.45 103.8)
-		(end 122.4 103.8)
-		(width 0.3)
-		(locked yes)
+		(start 118.562 103.784)
+		(end 119.3 103.784)
+		(width 0.4)
 		(layer "F.Cu")
 		(net 3)
 	)
 	(segment
-		(start 73.7494 71.3014)
-		(end 73.7494 70.7136)
-		(width 0.15)
+		(start 106.154 59.292)
+		(end 112.222 59.292)
+		(width 0.4)
 		(layer "F.Cu")
 		(net 3)
 	)
 	(segment
-		(start 113.2037 60.2737)
-		(end 113.2037 60.4999)
-		(width 0.15)
+		(start 113.55 60.846)
+		(end 113.848 61.144)
+		(width 0.4)
 		(layer "F.Cu")
 		(net 3)
 	)
 	(segment
-		(start 118.5621 103.7843)
-		(end 118.7076 103.9298)
+		(start 73.7494 71.3014)
+		(end 73.7494 70.7136)
 		(width 0.15)
 		(layer "F.Cu")
@@
 	)
 	(segment
-		(start 100.8627 54.1)
-		(end 106.0545 59.2918)
-		(width 0.15)
+		(start 70.75 54.1)
+		(end 60.6 54.1)
+		(width 0.4)
 		(layer "F.Cu")
 		(net 3)
@@
 	)
 	(segment
-		(start 68 67)
-		(end 61.602 67)
-		(width 0.15)
+		(start 119.5 103.975)
+		(end 121.225 103.975)
+		(width 0.4)
 		(layer "F.Cu")
 		(net 3)
 	)
 	(segment
-		(start 112.2218 59.2918)
-		(end 113.2037 60.2737)
-		(width 0.15)
+		(start 100.962 54.1)
+		(end 106.154 59.292)
+		(width 0.4)
 		(layer "F.Cu")
 		(net 3)
 	)
 	(segment
-		(start 121.225 103.975)
-		(end 121.45 103.8)
-		(width 0.3)
-		(locked yes)
+		(start 113.55 59.942)
+		(end 113.55 60.846)
+		(width 0.4)
+		(layer "F.Cu")
+		(net 3)
+	)
+	(segment
+		(start 70.175 70.05)
+		(end 69.225 71)
+		(width 0.4)
 		(layer "F.Cu")
 		(net 3)
@@
 	)
 	(segment
-		(start 72.8625 70.05)
-		(end 70.175 70.05)
-		(width 0.15)
+		(start 118.562 104.45)
+		(end 119.25 104.2)
+		(width 0.4)
 		(layer "F.Cu")
 		(net 3)
 	)
 	(segment
-		(start 113.2037 60.4999)
-		(end 113.8476 61.1438)
+		(start 73.7494 70.7136)
+		(end 73.0858 70.05)
 		(width 0.15)
 		(layer "F.Cu")
@@
 	)
 	(segment
-		(start 73.7494 70.7136)
-		(end 73.0858 70.05)
-		(width 0.15)
+		(start 70.175 69.175)
+		(end 70.175 70.05)
+		(width 0.4)
 		(layer "F.Cu")
 		(net 3)
 	)
 	(segment
-		(start 106.0545 59.2918)
-		(end 112.2218 59.2918)
-		(width 0.15)
+		(start 70.75 54.1)
+		(end 100.962 54.1)
+		(width 0.4)
 		(layer "F.Cu")
 		(net 3)
 	)
 	(segment
-		(start 60.8114 54.1)
-		(end 70.75 54.1)
-		(width 0.15)
+		(start 60.6 54.1)
+		(end 58.8 55.9)
+		(width 0.4)
 		(layer "F.Cu")
 		(net 3)
 	)
 	(segment
-		(start 61.602 67)
-		(end 58.9717 64.3697)
-		(width 0.15)
+		(start 112.222 59.292)
+		(end 112.9 59.292)
+		(width 0.4)
 		(layer "F.Cu")
 		(net 3)
 	)
 	(segment
-		(start 70.175 70.05)
-		(end 69.225 71)
-		(width 0.15)
+		(start 121.45 103.8)
+		(end 122.4 103.8)
+		(width 0.4)
 		(layer "F.Cu")
 		(net 3)
@@
 		(net 3)
 	)
+	(via
+		(at 118.562 104.45)
+		(size 0.45)
+		(drill 0.2)
+		(layers "F.Cu" "B.Cu")
+		(net 3)
+	)
 	(segment
-		(start 118.5621 80.1575)
-		(end 118.5621 103.7843)
-		(width 0.15)
+		(start 113.848 75.443)
+		(end 118.3 79.895)
+		(width 0.4)
 		(layer "B.Cu")
 		(net 3)
 	)
 	(segment
-		(start 113.8476 61.1438)
-		(end 113.8476 75.443)
-		(width 0.15)
+		(start 118.3 103.522)
+		(end 118.562 103.784)
+		(width 0.4)
 		(layer "B.Cu")
 		(net 3)
 	)
 	(segment
-		(start 113.8476 75.443)
-		(end 118.5621 80.1575)
-		(width 0.15)
+		(start 118.562 103.784)
+		(end 118.562 104.45)
+		(width 0.4)
+		(layer "B.Cu")
+		(net 3)
+	)
+	(segment
+		(start 118.3 79.895)
+		(end 118.3 103.522)
+		(width 0.4)
+		(layer "B.Cu")
+		(net 3)
+	)
+	(segment
+		(start 113.848 61.144)
+		(end 113.848 75.443)
+		(width 0.4)
 		(layer "B.Cu")
 		(net 3)
@@
 	)
 	(segment
-		(start 94.848008 66.448008)
-		(end 95.45 66.599999)
-		(width 0.2)
-		(layer "F.Cu")
-		(net 10)
-	)
-	(segment
 		(start 97.175 76.7)
 		(end 97.975 76.7)
@@
 	)
 	(segment
+		(start 94.848 66.447999)
+		(end 95.343 66.943)
+		(width 0.2)
+		(layer "F.Cu")
+		(net 10)
+	)
+	(segment
 		(start 87 91.45)
 		(end 87.82 91.45)
@@
 	)
 	(via
-		(at 67.798333 56.1239)
+		(at 87.8765 84.6174)
 		(size 0.45)
 		(drill 0.2)
@@
 	)
 	(via
-		(at 87.8765 84.6174)
+		(at 90.95 93.95)
 		(size 0.45)
 		(drill 0.2)
@@
 	)
 	(via
-		(at 90.95 93.95)
+		(at 95.343 66.943)
 		(size 0.45)
 		(drill 0.2)
@@
 		(size 0.45)
 		(drill 0.2)
-		(layers "F.Cu" "B.Cu")
-		(net 10)
-	)
-	(via
-		(at 95.45 66.599999)
-		(size 0.45)
-		(drill 0.2)
