File: hardware/airnote.kicad_sch (KiCad schematic)
At the start: 26 parts, among them J2 SWD 3V3 GND DIO CLK RUN, SW1 BOOTSEL, SW2 RESET, U1 RP2040, U2 W25Q16JVSSIQ, Y1 12MHz ABM8-272-T3

Commit message: Phase 2: rev 0.2 layout with coupled USB pair, crystal/IOVDD fixes and JLC sourcing
Hardware (implementer, verified by overseer):
- Stackup set to JLC04161H-7628. USB_DIFF net class at 0.25/0.15 mm; all six
  USB nets on F.Cu with no vias over continuous In1 GND.
- Crystal moved under U1: XIN 4.1 mm with no vias (was 7.8 mm, 2 vias).
  IOVDD pin 22 to C6 2.9 mm (was 6.1 mm).
- airnote.kicad_dru values now carry units. KiCad had been discarding the
  unitless file, so its rules were never enforced. DRC still passes.
- U2 corrected to W25Q16JVSNIQ (150-mil, matches footprint). J1, RV1, J2 and
  passives switched to in-stock JLC/LCSC parts. LCSC numbers in the schematic,
  footprints and bom.csv.
- Three global fiducials. ERC 0, DRC 0, parity 0; outputs regenerated.

Docs: fabrication plan, requirements, README, assembly brief and bring-up
updated for rev 0.2. Surface finish recorded as an order-time decision.
Parts:
- C1, C2: LCSC (none) -> C1644; MPN GRM1885C1H150JA01D -> CL10C150JB8NNNC
- C10, C11, C12, C15, C3, C4, C5, C6, C7, C8, C9: LCSC (none) -> C14663; MPN GRM188R71C104KA01D -> CC0603KRX7R9BB104
- C13, C14: LCSC (none) -> C15849; MPN GRM188R71A105KA61D -> CL10A105KB8NNNC
- J2: LCSC (none) -> C32713271; MPN TSW-105-07-G-S -> HX PZ2.54-1x5P ZZ
- R1, R3: LCSC (none) -> C21190; MPN RC0603FR-071KL -> 0603WAF1001T5E
- R2, R4: LCSC (none) -> C25804; MPN RC0603FR-0710KL -> 0603WAF1002T5E
- R5: LCSC (none) -> C22936; MPN RC0603FR-071RL -> 0603WAF100KT5E
- SW1, SW2: LCSC (none) -> C2886898
- U1: LCSC (none) -> C2040
- U2: value W25Q16JVSSIQ -> W25Q16JVSNIQ; LCSC (none) -> C2456211; MPN W25Q16JVSSIQ -> W25Q16JVSNIQ
- Y1: LCSC (none) -> C20625731
