File: hardware/instrument.kicad_sch (KiCad schematic)
At the start: 21 parts, among them J3 SPEAKER 8ohm >=1W, SW3 MUTE / PLAY, U4 VL53L1CXV0FY/1, U5 MAX98357AETE+T

Commit message: Phase 2: rev 0.2 layout with coupled USB pair, crystal/IOVDD fixes and JLC sourcing
Hardware (implementer, verified by overseer):
- Stackup set to JLC04161H-7628. USB_DIFF net class at 0.25/0.15 mm; all six
  USB nets on F.Cu with no vias over continuous In1 GND.
- Crystal moved under U1: XIN 4.1 mm with no vias (was 7.8 mm, 2 vias).
  IOVDD pin 22 to C6 2.9 mm (was 6.1 mm).
- airnote.kicad_dru values now carry units. KiCad had been discarding the
  unitless file, so its rules were never enforced. DRC still passes.
- U2 corrected to W25Q16JVSNIQ (150-mil, matches footprint). J1, RV1, J2 and
  passives switched to in-stock JLC/LCSC parts. LCSC numbers in the schematic,
  footprints and bom.csv.
- Three global fiducials. ERC 0, DRC 0, parity 0; outputs regenerated.

Docs: fabrication plan, requirements, README, assembly brief and bring-up
updated for rev 0.2. Surface finish recorded as an order-time decision.
Parts:
- C19, C21, C23: LCSC (none) -> C14663; MPN GRM188R71C104KA01D -> CC0603KRX7R9BB104
- C20, C22: LCSC (none) -> C1779; MPN GRM21BR71A475KA73L -> CL21A475KAQNNNE
- D2: LCSC (none) -> C125094
- J3: LCSC (none) -> C131337
- R10, R11, R14, R16: LCSC (none) -> C25804; MPN RC0603FR-0710KL -> 0603WAF1002T5E
- R12, R13: LCSC (none) -> C23186; MPN RC0603FR-075K1L -> 0603WAF5101T5E
- R15: LCSC (none) -> C25803; MPN RC0603FR-07100KL -> 0603WAF1003T5E
- R17, R18: LCSC (none) -> C21190; MPN RC0603FR-071KL -> 0603WAF1001T5E
- R19: LCSC (none) -> C22935; MPN RC0603FR-071ML -> 0603WAF1004T5E
- RV1: LCSC (none) -> C5710902; MPN PTV09A-1020F-B103 -> PTV09A-4015F-B103
- SW3: LCSC (none) -> C221665
- U4: LCSC (none) -> C190004
- U5: LCSC (none) -> C910544
