File: hardware/power.kicad_sch (KiCad schematic)
At the start: 22 parts, among them J1 USB-C USB2.0, U3 AP2112K-3.3

Commit message: Phase 2: rev 0.2 layout with coupled USB pair, crystal/IOVDD fixes and JLC sourcing
Hardware (implementer, verified by overseer):
- Stackup set to JLC04161H-7628. USB_DIFF net class at 0.25/0.15 mm; all six
  USB nets on F.Cu with no vias over continuous In1 GND.
- Crystal moved under U1: XIN 4.1 mm with no vias (was 7.8 mm, 2 vias).
  IOVDD pin 22 to C6 2.9 mm (was 6.1 mm).
- airnote.kicad_dru values now carry units. KiCad had been discarding the
  unitless file, so its rules were never enforced. DRC still passes.
- U2 corrected to W25Q16JVSNIQ (150-mil, matches footprint). J1, RV1, J2 and
  passives switched to in-stock JLC/LCSC parts. LCSC numbers in the schematic,
  footprints and bom.csv.
- Three global fiducials. ERC 0, DRC 0, parity 0; outputs regenerated.

Docs: fabrication plan, requirements, README, assembly brief and bring-up
updated for rev 0.2. Surface finish recorded as an order-time decision.
Parts:
- C16, C17: LCSC (none) -> C15849; MPN GRM188R71A105KA61D -> CL10A105KB8NNNC
- C18: LCSC (none) -> C14663; MPN GRM188R71C104KA01D -> CC0603KRX7R9BB104
- D1: LCSC (none) -> C7519
- F1: LCSC (none) -> C163512
- J1: LCSC (none) -> C5184243; MPN USB4105-GF-A -> USB4105-GF-A-120
- R6, R7: LCSC (none) -> C23186; MPN RC0603FR-075K1L -> 0603WAF5101T5E
- R8, R9: LCSC (none) -> C25190; MPN RC0603FR-0727RL -> 0603WAF270JT5E
- U3: LCSC (none) -> C51118
